File: pcbee.kicad_pcb (KiCad board)
At the start: 2 copper layers, 50.8 x 43.2 mm, 5 parts

Commit message: Rev C intial design work
Parts:
- removed the G*** at (150.5, 94.6)
- removed REF**: MountingHole_2.2mm_M2_Pad, Mounting_Holes:MountingHole_2.2mm_M2_Pad
- added C1: 12pF, Capacitors_SMD:C_0603_HandSoldering, B.Cu at (162.0, 84.6)
- added C2: 12pF, Capacitors_SMD:C_0603_HandSoldering, B.Cu at (161.1, 77.3)
- added C3: 1u, Capacitors_SMD:C_0805_HandSoldering, B.Cu at (158.8, 95.4)
- added D3: RED, LEDs:LED_0805_HandSoldering, F.Cu at (149.9, 114.3)
- added G***: LOGO, custom:bee, F.Cu at (150.5, 96.5)
- added J2: USB_B_Micro, Connectors_USB:USB_Micro-B_Molex_47346-0001, B.Cu at (133.1, 85.3)
- added R1: 330, Resistors_SMD:R_0603_HandSoldering, B.Cu at (165.1, 89.5)
- added R10: 470, Resistors_SMD:R_0603_HandSoldering, B.Cu at (162.6, 94.2)
- added R11: 100k, Resistors_SMD:R_0603_HandSoldering, B.Cu at (165.1, 86.1)
- added R12: 100k, Resistors_SMD:R_0603_HandSoldering, B.Cu at (155.9, 93.0)
- added R2: 330, Resistors_SMD:R_0603_HandSoldering, B.Cu at (165.1, 87.9)
- added R3: 330, Resistors_SMD:R_0603_HandSoldering, B.Cu at (165.1, 91.1)
- added R4: 330, Resistors_SMD:R_0603_HandSoldering, B.Cu at (134.4, 95.1)
- added R5: 330, Resistors_SMD:R_0603_HandSoldering, B.Cu at (134.4, 96.6)
- added R6: 330, Resistors_SMD:R_1206_HandSoldering, B.Cu at (138.7, 87.7)
- added R7: 10k, Resistors_SMD:R_0603_HandSoldering, B.Cu at (138.1, 80.3)
- added R8: 22, Resistors_SMD:R_0603_HandSoldering, B.Cu at (142.6, 86.4)
- added R9: 22, Resistors_SMD:R_0603_HandSoldering, B.Cu at (142.6, 87.9)
- added SW1: SW_SPDT, Buttons_Switches_SMD:SW_SPDT_PCM12, B.Cu at (131.8, 104.1)
- added SW2: RIGHT, Buttons_Switches_SMD:SW_SPST_B3U-1000P, B.Cu at (168.9, 96.5)
- added SW3: LEFT, Buttons_Switches_SMD:SW_SPST_B3U-1000P, B.Cu at (130.3, 96.5)
- added TP1: Vdd, Connectors_TestPoints:Test_Point_Pad_1.0x1.0mm, B.Cu at (159.7, 90.7)
- added TP2: MISO, Connectors_TestPoints:Test_Point_Pad_1.0x1.0mm, B.Cu at (142.7, 78.8)
- added TP3: MOSI, Connectors_TestPoints:Test_Point_Pad_1.0x1.0mm, B.Cu at (142.7, 82.1)
- added TP4: CLK, Connectors_TestPoints:Test_Point_Pad_1.0x1.0mm, B.Cu at (142.7, 83.8)
- added TP5: RST, Connectors_TestPoints:Test_Point_Pad_1.0x1.0mm, B.Cu at (139.1, 78.7)
- added TP6: GND, Connectors_TestPoints:Test_Point_Pad_1.0x1.0mm, B.Cu at (139.2, 76.8)
- added U1: ATmega32U4-AU, Housings_QFP:TQFP-44_10x10mm_Pitch0.8mm, B.Cu at (151.8, 84.5)
- added Y1: 16MHz, Crystals:Crystal_SMD_3225-4pin_3.2x2.5mm_HandSoldering, B.Cu at (161.3, 81.1)
- BT1: footprint Battery_Holders:Keystone_103_1x20mm-CoinCell -> Battery_Holders:Keystone_3034_1x20mm-CoinCell
- D1, D2: value LED -> ASMB-KTF0-0A306; footprint LEDs:LED_D5.0mm -> custom:ASMB-KTF0-0A306; moved to F.Cu
- moved BT1 11.0 mm to (149.9, 107.3)
- moved D1 3.95 mm to (169.3, 94.5)
- moved D2 3.86 mm to (130.5, 94.5)
Connections:
- BT1 pad 2: Net-(BT1-Pad2) -> GND
- D1 pad 1: Net-(BT1-Pad2) -> VDD
- D1 pad 2: Net-(BT1-Pad1) -> Net-(D1-Pad2)
- D2 pad 1: Net-(BT1-Pad2) -> VDD
- D2 pad 2: Net-(BT1-Pad1) -> Net-(D2-Pad2)
Routing:
- net VDD: track 0.00 -> 126.8 mm, vias 0 -> 2
- net GND: track 0.00 -> 83.5 mm, vias 0 -> 4
- net Net-(BT1-Pad2): track 56.7 -> 0.00 mm
- net Net-(R12-Pad1): track 0.00 -> 30.1 mm
- net Net-(R4-Pad2): track 0.00 -> 28.6 mm, vias 0 -> 2
- net Net-(R5-Pad2): track 0.00 -> 27.8 mm, vias 0 -> 2
- net Net-(R6-Pad2): track 0.00 -> 25.0 mm, vias 0 -> 2
- net Net-(D3-Pad2): track 0.00 -> 24.6 mm, vias 0 -> 1
- net Net-(R11-Pad1): track 0.00 -> 20.9 mm
- net Net-(D2-Pad4): track 0.00 -> 17.5 mm, vias 0 -> 1
- net Net-(C1-Pad1): track 0.00 -> 16.5 mm
- net Net-(BT1-Pad1): track 66.6 -> 50.5 mm
- net Net-(C2-Pad1): track 0.00 -> 15.9 mm
- net Net-(J2-Pad1): track 0.00 -> 15.6 mm
- net Net-(D1-Pad3): track 0.00 -> 13.4 mm, vias 0 -> 1
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- added copper zone on B.Cu, net GND
- added copper zone on F.Cu, net GND
- removed copper zone on F.Cu, net (none)
Other:
- net class Default: clearance 0.2 -> 0.1524; trace_width 0.55 -> 0.1524; via_dia 0.6 -> 0.508; via_drill 0.4 -> 0.3048
- rule trace_clearance: 0.2 -> 0.1524
- rule trace_min: 0.2 -> 0.1524
- rule via_min_drill: 0.3 -> 0.3048
- rule via_min_size: 0.4 -> 0.508
- board text removed: "Designed by Committee at Hackspace Manchester 2018"
