File: pcbee.sch (KiCad schematic (older format))
At the start: 3 parts

Commit message: Rev C intial design work
Parts:
- removed D1, D2: LED, LEDs:LED_D5.0mm, symbol LED
- added C1, C2: 12pF, Capacitors_SMD:C_0603_HandSoldering, symbol Device:C
- added C3: 1u, Capacitors_SMD:C_0805_HandSoldering, symbol Device:C
- added D1, D2: ASMB-KTF0-0A306, custom:ASMB-KTF0-0A306, symbol Device:LED_ARGB
- added D3: RED, LEDs:LED_0805_HandSoldering, symbol Device:LED
- added J2: USB_B_Micro, Connectors_USB:USB_Micro-B_Molex_47346-0001, symbol Connector:USB_B_Micro
- added R1, R2, R3, R4, R5: 330, Resistors_SMD:R_0603_HandSoldering, symbol Device:R
- added R10: 470, Resistors_SMD:R_0603_HandSoldering, symbol Device:R
- added R11, R12: 100k, Resistors_SMD:R_0603_HandSoldering, symbol Device:R
- added R6: 330, Resistors_SMD:R_1206_HandSoldering, symbol Device:R
- added R7: 10k, Resistors_SMD:R_0603_HandSoldering, symbol Device:R
- added R8, R9: 22, Resistors_SMD:R_0603_HandSoldering, symbol Device:R
- added SW1: SW_SPDT, Buttons_Switches_SMD:SW_SPDT_PCM12, symbol Switch:SW_SPDT
- added SW2: RIGHT, Buttons_Switches_SMD:SW_SPST_B3U-1000P, symbol Switch:SW_Push
- added SW3: LEFT, Buttons_Switches_SMD:SW_SPST_B3U-1000P, symbol Switch:SW_Push
- added TP1: Vdd, Connectors_TestPoints:Test_Point_Pad_1.0x1.0mm, symbol Connector:Test_Point
- added TP2: MISO, Connectors_TestPoints:Test_Point_Pad_1.0x1.0mm, symbol Connector:Test_Point
- added TP3: MOSI, Connectors_TestPoints:Test_Point_Pad_1.0x1.0mm, symbol Connector:Test_Point
- added TP4: CLK, Connectors_TestPoints:Test_Point_Pad_1.0x1.0mm, symbol Connector:Test_Point
- added TP5: RST, Connectors_TestPoints:Test_Point_Pad_1.0x1.0mm, symbol Connector:Test_Point
- added TP6: GND, Connectors_TestPoints:Test_Point_Pad_1.0x1.0mm, symbol Connector:Test_Point
- added U1: ATmega32U4-AU, Housings_QFP:TQFP-44_10x10mm_Pitch0.8mm, symbol MCU_Microchip_ATmega:ATmega32U4-AU
- added Y1: 16MHz, Crystals:Crystal_SMD_3225-4pin_3.2x2.5mm_HandSoldering, symbol Device:Crystal_GND24
- BT1: footprint Battery_Holders:Keystone_103_1x20mm-CoinCell -> Battery_Holders:Keystone_3034_1x20mm-CoinCell; symbol Battery_Cell -> pcbee-rescue:Battery_Cell
Connections:
- net labels added: GND, LED, RST, VDD
- wire segments 2 -> 116
- no-connect marks 0 -> 3
Other:
- note added: "IND LED 13\n"
- note added: "LEFT\nR \nG \nB"
- note added: "RIGHT\nR \nG \nB"
- moved on the sheet: BT1
